File: OBS-buttons-panel.sch (EAGLE design)
At the start: 23 parts

Commit message: initial prototype
Parts:
- removed BOARD2: (no value), SPCoast:BOARD100X50-NOHOLES
- removed CON1: (no value), SPCoast:CONNECTOR-M02508-LOCK
- removed J1, J2, J3, J4: (no value), SPCoast:CONNECTOR-M08LOCK
- removed LED1, LED2, LED3, LED4, LED5, LED6: (no value), SPCoast:LEDLED5MM
- removed R1, R2, R3, R4, R5, R6: (no value), SPCoast:RPTH04
- removed SW1, SW2, SW3: (no value), SPCoast:SWITCH-SPSTPTH-508
- removed U$1: ARDUINO-PRO-MICROEBAY, SPCoast:ARDUINO-PRO-MICROEBAY
Connections:
- removed net CUT: J1.3, SW1.O
- removed net CUT-LED: J2.1, R1.1
- removed net FADE: J1.4, SW1.S
- removed net FADE-LED: J2.6, R2.1
- removed net GND: CON1.A, J2.7, J2.8, J4.7, J4.8, SW1.P, SW2.P, SW3.P, U$1.GND, U$1.GND@2, U$1.GND@3
- removed net I1: J3.5, U$1.A0
- removed net I2: J3.4, U$1.D13
- removed net I3: J3.3, U$1.D12
- removed net I4: J3.2, U$1.D11
- removed net I5: J3.6, U$1.D8
- removed net I6: J3.7, U$1.D4
- removed net I7: J3.8, U$1.D2-SDA
- removed net N$1: LED1.C, R1.2
- removed net N$2: LED2.C, R2.2
- removed net N$3: LED3.C, R3.2
- removed net N$4: LED4.C, R4.2
- removed net N$5: LED5.C, R5.2
- removed net N$6: LED6.C, R6.2
- removed net O1: J4.1, U$1.*D3-SCL
- removed net O2: J4.2, U$1.*D5
- removed net O3: J4.3, U$1.*D6
- removed net O4: J4.4, U$1.D7
- removed net O5: J4.5, U$1.*D9
- removed net O6: J4.6, U$1.*D10
- removed net SCENE1: J1.5, SW2.O
- removed net SCENE1-LED: J2.2, R3.1
- removed net SCENE2: J1.6, SW2.S
- removed net SCENE2-LED: J2.5, R4.1
- removed net SCENE3: J1.7, SW3.O
- removed net SCENE3-LED: J2.3, R5.1
- removed net SCENE4: J1.8, SW3.S
- removed net SCENE4-LED: J2.4, R6.1
- removed net TRANSITION: CON1.B, J1.2
- removed net VCC: J1.1, J3.1, LED1.A, LED2.A, LED3.A, LED4.A, LED5.A, LED6.A, U$1.VCC
